File: eagle/midi_thru.sch (EAGLE design)
At the start: 24 parts, among them IC2 40106N

Commit message: routed
Parts:
- added JP1: (no value), jumper:JP1E
- R10, R11, R13, R14, R15, R2, R3, R4, R6, R7, R9: device rcl:R-US_0207/10 -> rcl:R-US_0207/7
- renumbered U$1 to THRU_1, U$2 to THRU_2, U$3 to THRU_3, U$4 to THRU_4, U$5 to IN
Connections:
- removed net N$22: IC2B.O, R6.1
- removed net N$24: IC2D.O, R9.1
- removed net N$25: IC2E.O, R10.1
- new net N$5: IC2D.O, R10.1
- new net N$8: IC2E.O, R9.1
- new net N$9: IC2F.O, R6.1
- net +5V: now also JP1.2
- net GND: now also ING$2.MT, ING$3.MT, ING$4.MT, ING$5.MT, THRU_1G$2.MT, THRU_1G$3.MT, THRU_1G$4.MT, THRU_1G$5.MT, THRU_2G$2.MT, THRU_2G$3.MT, THRU_2G$4.MT, THRU_2G$5.MT, THRU_3G$2.MT, THRU_3G$3.MT, THRU_3G$4.MT, THRU_3G$5.MT, THRU_4G$2.MT, THRU_4G$3.MT, THRU_4G$4.MT, THRU_4G$5.MT
- net N$2: now also IC2B.O; no longer IC2F.O
- net N$35: now also THRU_3G$1.4
- net N$6: now also JP1.1
Other:
- note removed: "MIDI_IN_4"
- note removed: "MIDI_IN_5"
- moved on the sheet: IC2B, IC2D, IC2E, IC2F
