File: eagle/midi_thru.brd (EAGLE design)
At the start: 100.8 x 80.8 mm, 25 parts, among them IC2 40106N

Commit message: first cut happened
Parts:
- moved R13 16.6 mm to (27.9, 20.3)
- moved R14 10.6 mm to (69.1, 17.3), turned to 90 degrees
- moved LED1 9.92 mm to (61.0, 24.1)
- moved R9 7.41 mm to (85.1, 33.0), turned to 270 degrees
- moved R11 5.24 mm to (20.3, 20.3), turned to 0 degrees
- moved D1 4.02 mm to (52.1, 38.1)
- moved R6 4.02 mm to (64.8, 40.6)
- moved R10 3.70 mm to (81.5, 24.4), turned to 180 degrees
- moved R15 3.61 mm to (89.9, 18.8), turned to 0 degrees
- moved C2 2.84 mm to (30.5, 27.9)
- moved OK1 2.84 mm to (52.1, 29.2)
- moved R2 2.84 mm to (43.2, 33.0)
- moved C1 2.84 mm to (26.7, 27.9)
- moved IC2 2.54 mm to (71.1, 33.0)
- moved 78L05 2.54 mm to (36.8, 27.9), turned to 0 degrees
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Routing:
- net N$23: track 111.2 -> 44.5 mm
- net GND: track 245.2 -> 292.3 mm
- net +5V: track 129.3 -> 154.5 mm
- net N$34: track 4.52 -> 27.2 mm
- net N$30: track 34.1 -> 49.2 mm, vias 2 -> 0
- net N$8: track 3.16 -> 14.6 mm
- net N$5: track 4.95 -> 16.0 mm
- net N$28: track 70.7 -> 62.0 mm
- net N$35: track 15.1 -> 6.97 mm
- net N$26: track 75.7 -> 79.5 mm
- net N$7: track 15.2 -> 18.2 mm
- net N$27: track 5.23 -> 7.09 mm
- net N$33: track 5.14 -> 6.57 mm
- net N$6: track 37.8 -> 39.2 mm
- net N$4: track 5.41 -> 4.19 mm
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Other:
- outline, holes or cut-outs redrawn
